Commit message: Simplified model using merged links

File: umrt-project-perry-description/urdf/robot.urdf (robot description, URDF)
Before this commit: robot pp-arm, 6 links, 5 joints
Links:
- link flat_pattern_of_plate_1: geometry collision mesh filename=package://assets/merged/flat_pattern_of_plate_1_collision.s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; visual mesh filename=package://assets/merged/flat_pattern_of_plate_1_visual.stl
- link part_33: geometry collision mesh filename=package://assets/merged/part_33_collision.stl; visual mesh filename=package://assets/merged/part_33_visual.stl
- link part_43: geometry collision mesh filename=package://assets/merged/part_43_collision.stl; visual mesh filename=package://assets/merged/part_43_visual.stl
- link part_48: geometry collision mesh filename=package://assets/merged/part_48_collision.stl; visual mesh filename=package://assets/merged/part_48_visual.stl
- link part_6: geometry collision mesh filename=package://assets/merged/part_6_collision.stl; visual mesh filename=package://assets/merged/part_6_visual.stl
- link part_8: geometry collision mesh filename=package://assets/merged/part_8_collision.stl; visual mesh filename=package://assets/merged/part_8_visual.stl
