Commit message: Pasted new URDF into xacro

File: umrt-project-perry-description/urdf/project_perry_description.urdf.xacro (robot description, xacro)
@@ -2,240 +2,194 @@
 <robot xmlns:xacro="http://www.ros.org/wiki/xacro">
     <xacro:macro name="project_perry" params="parent prefix *origin">
-        <!-- Constants for robot dimensions -->
-        <xacro:property name="mass" value="1"/> <!-- arbitrary value for mass -->
-        <xacro:property name="base_width" value="1"/>
-        <xacro:property name="base_height" value="0.6"/>
-        <xacro:property name="platter_radius" value="0.75"/>
-        <xacro:property name="platter_height" value="0.1"/>
-        <xacro:property name="width" value="0.1"/> <!-- Square dimensions (widthxwidth) of beams -->
-        <xacro:property name="height1" value="2"/> <!-- Link 1 -->
-        <xacro:property name="height2" value="1"/> <!-- Link 2 -->
-        <xacro:property name="height3" value="1"/> <!-- Link 3 -->
-        <xacro:property name="gripper_width" value="0.4"/>
-        <xacro:property name="gripper_breadth" value="0.1"/>
-        <xacro:property name="gripper_thickness" value="0.05"/>
-        <xacro:property name="finger_length" value="0.2"/>
-        <xacro:property name="finger_thickness" value="0.05"/>
-        <xacro:property name="axel_offset" value="0.05"/> <!-- Space btw top of beam and the each joint -->
         <joint name="${prefix}base_joint" type="fixed">
             <xacro:insert_block name="origin"/>
             <parent link="${parent}"/>
-            <child link="${prefix}base_link"/>
+            <child link="part_48"/>
         </joint>
-        <!-- Base Link -->
-        <link name="${prefix}base_link">
+        <!-- Generated using onshape-to-robot -->
+        <!-- Link part_48 -->
+        <link name="part_48">
+            <inertial>
+            <origin xyz="0.00286812 -0.0209097 0.0286943" rpy="0 0 0"/>
+            <mass value="2.80632"/>
+            <inertia ixx="0.0231691" ixy="0.00065571" ixz="-0.000230556" iyy="0.0147789" iyz="0.000656447" izz="0.0344912"/>
+            </inertial>
+            <!-- Part part_48_parts -->
+            <visual>
+            <origin xyz="0.00286812 -0.0209097 0.0286943" rpy="0 -0 0"/>
+            <geometry>
+                <mesh filename="package://assets/merged/part_48_visual.stl"/>
+            </geometry>
+            <material name="part_48_parts_material">
+                <color rgba="0.0745098 0.678431 0.972549 1"/>
+            </material>
+            </visual>
             <collision>
-                <origin xyz="0 0 ${base_height/2}" rpy="0 0 0"/>
-                <geometry>
-                    <box size="${base_width} ${base_width} ${base_height}"/>
-                </geometry>
+            <origin xyz="0.00286812 -0.0209097 0.0286943" rpy="0 -0 0"/>
+            <geometry>
+                <mesh filename="package://assets/merged/part_48_collision.stl"/>
+            </geometry>
             </collision>
+        </link>
+        <!-- Link part_43 -->
+        <link name="part_43">
+            <inertial>
+            <origin xyz="-0.0119595 -0.00118557 -0.0231327" rpy="0 0 0"/>
+            <mass value="1.84265"/>
+            <inertia ixx="0.00590316" ixy="0.000138602" ixz="-0.000532603" iyy="0.00955076" iyz="2.11489e-05" izz="0.012905"/>
+            </inertial>
+            <!-- Part part_43_parts -->
             <visual>
-                <origin xyz="0 0 ${base_height/2}" rpy="0 0 0"/>
-                <geometry>
-                    <box size="${base_width} ${base_width} ${base_height}"/>
-                </geometry>
-                <material name="orange"/>
+            <origin xyz="-0.0119595 -0.00118557 -0.0231327" rpy="-3.13855 -0.016189 -0.393062"/>
+            <geometry>
+                <mesh filename="package://assets/merged/part_43_visual.stl"/>
+            </geometry>
+            <material name="part_43_parts_material">
+                <color rgba="0.570634 0.573152 0.433741 1"/>
+            </material>
             </visual>
+            <collision>
+            <origin xyz="-0.0119595 -0.00118557 -0.0231327" rpy="-3.13855 -0.016189 -0.393062"/>
+            <geometry>
+                <mesh filename="package://assets/merged/part_43_collision.stl"/>
+            </geometry>
+            </collision>
+        </link>
+        <!-- Link part_33 -->
+        <link name="part_33">
             <inertial>
-                <origin xyz="0 0 ${base_height/2}" rpy="0 0 0"/>
-                <mass value="${mass}"/>
-                <inertia
-                        ixx="${mass / 12.0 * (base_width*base_width + base_height*base_height)}" ixy="0.0" ixz="0.0"
-                        iyy="${mass / 12.0 * (base_height*base_height + base_width*base_width)}" iyz="0.0"
-                        izz="${mass / 12.0 * (base_width*base_width + base_width*base_width)}"/>
+            <origin xyz="0.191821 -0.0003306 -0.0214358" rpy="0 0 0"/>
+            <mass value="2.10608"/>
+            <inertia ixx="0.00610007" ixy="-0.00133336" ixz="-0.000268934" iyy="0.0355323" iyz="-2.46829e-05" izz="0.0374741"/>
             </inertial>
+            <!-- Part part_33_parts -->
+            <visual>
+            <origin xyz="0.191821 -0.0003306 -0.0214358" rpy="1.61286 1.17742 1.48782"/>
+            <geometry>
+                <mesh filename="package://assets/merged/part_33_visual.stl"/>
+            </geometry>
+            <material name="part_33_parts_material">
+                <color rgba="0.470126 0.661547 0.742536 1"/>
+            </material>
+            </visual>
+            <collision>
+            <origin xyz="0.191821 -0.0003306 -0.0214358" rpy="1.61286 1.17742 1.48782"/>
+            <geometry>
+                <mesh filename="package://assets/merged/part_33_collision.stl"/>
+            </geometry>
+            </collision>
         </link>
-        <joint name="${prefix}base_yaw_joint" type="continuous">
-            <parent link="${prefix}base_link"/>
-            <child link="${prefix}shoulder_link"/>
-            <origin xyz="0 0 ${base_height - axel_offset}" rpy="0 0 0"/>
+        <!-- Link flat_pattern_of_plate_1 -->
+        <link name="flat_pattern_of_plate_1">
+            <inertial>
+            <origin xyz="0.0157793 -0.119702 0.0450796" rpy="0 0 0"/>
+            <mass value="2.41986"/>
+            <inertia ixx="0.06464" ixy="0.0122868" ixz="-5.92337e-06" iyy="0.0115771" iyz="2.1658e-05" izz="0.0644214"/>
+            </inertial>
+            <!-- Part flat_pattern_of_plate_1_parts -->
+            <visual>
+            <origin xyz="0.0157793 -0.119702 0.0450796" rpy="1.61286 1.17742 -1.65378"/>
+            <geometry>
+                <mesh filename="package://assets/merged/flat_pattern_of_plate_1_visual.stl"/>
+            </geometry>
+            <material name="flat_pattern_of_plate_1_parts_material">
+                <color rgba="0.358967 0.586653 0.658572 1"/>
+            </material>
+            </visual>
+            <collision>
+            <origin xyz="0.0157793 -0.119702 0.0450796" rpy="1.61286 1.17742 -1.65378"/>
+            <geometry>
+                <mesh filename="package://assets/merged/flat_pattern_of_plate_1_collision.stl"/>
+            </geometry>
+            </collision>
+        </link>
+        <!-- Link part_6 -->
+        <link name="part_6">
+            <inertial>
+            <origin xyz="1.74216e-05 -0.0133229 -0.0449775" rpy="0 0 0"/>
+            <mass value="0.114952"/>
+            <inertia ixx="0.000141143" ixy="-3.67177e-10" ixz="8.43247e-07" iyy="0.000208967" iyz="4.47572e-13" izz="9.77212e-05"/>
+            </inertial>
+            <!-- Part part_6_parts -->
+            <visual>
+            <origin xyz="1.74216e-05 -0.0133229 -0.0449775" rpy="1.61286 1.17742 -1.4845"/>
+            <geometry>
+                <mesh filename="package://assets/merged/part_6_visual.stl"/>
+            </geometry>
+            <material name="part_6_parts_material">
+                <color rgba="0.0745098 0.678431 0.972549 1"/>
+            </material>
+            </visual>
+            <collision>
+            <origin xyz="1.74216e-05 -0.0133229 -0.0449775" rpy="1.61286 1.17742 -1.4845"/>
+            <geometry>
+                <mesh filename="package://assets/merged/part_6_collision.stl"/>
+            </geometry>
+            </collision>
+        </link>
+        <!-- Link part_8 -->
+        <link name="part_8">
+            <inertial>
+            <origin xyz="-7.09882e-18 1.30193e-17 -0.00183593" rpy="0 0 0"/>
+            <mass value="0.0230672"/>
+            <inertia ixx="6.54736e-06" ixy="-3.28523e-23" ixz="-1.16149e-21" iyy="6.54736e-06" iyz="-2.92654e-22" izz="1.27521e-05"/>
+            </inertial>
+            <!-- Part part_8_parts -->
+            <visual>
+            <origin xyz="-2.77556e-17 5.55112e-17 -0.00183593" rpy="-1.62212 0.391834 -2.8036"/>
+            <geometry>
+                <mesh filename="package://assets/merged/part_8_visual.stl"/>
+            </geometry>
+            <material name="part_8_parts_material">
+                <color rgba="0.972549 0.529412 0.00392157 1"/>
+            </material>
+            </visual>
+            <collision>
+            <origin xyz="-2.77556e-17 5.55112e-17 -0.00183593" rpy="-1.62212 0.391834 -2.8036"/>
+            <geometry>
+                <mesh filename="package://assets/merged/part_8_collision.stl"/>
+            </geometry>
+            </collision>
+        </link>
+        <!-- Joint from part_6 to part_8 -->
+        <joint name="wrist_roll" type="revolute">
+            <origin xyz="1.11022e-16 -0.0314483 -0.0449775" rpy="1.5708 -1.19705 3.14159"/>
+            <parent link="part_6"/>
+            <child link="part_8"/>
             <axis xyz="0 0 1"/>
-            <dynamics damping="0.7"/>
-            <limit effort="100" velocity="1.0"/>
+            <limit effort="10" velocity="10" lower="-3.141592653589793" upper="3.141592653589793"/>
         </joint>
-        <!-- Middle Link -->
-        <link name="${prefix}shoulder_link">
-            <collision>
-                <origin xyz="0 0 ${platter_height/2 + axel_offset}" rpy="0 0 0"/>
-                <geometry>
-                    <cylinder radius="${platter_radius}" length="${platter_height}"/>
-                </geometry>
-            </collision>
-            <visual>
-                <origin xyz="0 0 ${platter_height/2 + axel_offset}" rpy="0 0 0"/>
-                <geometry>
-                    <cylinder radius="${platter_radius}" length="${platter_height}"/>
-                </geometry>
-                <material name="yellow"/>
-            </visual>
-            <inertial>
-                <origin xyz="0 0 ${platter_height/2 - axel_offset}" rpy="0 0 0"/>
-                <mass value="${mass}"/>
-                <inertia
-                        ixx="${mass / 12.0 * (3*platter_radius*platter_radius + platter_height*platter_height)}"
-                        ixy="0.0" ixz="0.0"
-                        iyy="${mass / 12.0 * (3*platter_radius*platter_radius + platter_height*platter_height)}"
-                        iyz="0.0"
-                        izz="${mass / 2.0 * platter_radius*platter_radius}"/>
-            </inertial>
-        </link>
-        <joint name="${prefix}base_pitch_joint" type="revolute">
-            <parent link="${prefix}shoulder_link"/>
-            <child link="${prefix}humerus_link"/>
-            <origin xyz="0 0 ${platter_height + axel_offset*2}" rpy="0 0 0"/>
-            <axis xyz="0 1 0"/>
-            <dynamics damping="0.7"/>
-            <limit lower="${-pi/2.0}" upper="${pi/2.0}" effort="100" velocity="1.0"/>
+        <!-- Joint from flat_pattern_of_plate_1 to part_6 -->
+        <joint name="wrist_pitch" type="revolute">
+            <origin xyz="0.070773 -0.387287 0.0899558" rpy="8.40994e-16 7.19541e-16 -0.169273"/>
+            <parent link="flat_pattern_of_plate_1"/>
+            <child link="part_6"/>
+            <axis xyz="0 0 1"/>
+            <limit effort="10" velocity="10" lower="-1.22078" upper="1.92082"/>
         </joint>
-        <!-- Top Link -->
-        <link name="${prefix}humerus_link">
-            <collision>
-                <origin xyz="0 0 ${height3/2 - axel_offset}" rpy="0 0 0"/>
-                <geometry>
-                    <box size="${width} ${width} ${height3}"/>
-                </geometry>
-            </collision>
-            <visual>
-                <origin xyz="0 0 ${height3/2 - axel_offset}" rpy="0 0 0"/>
-                <geometry>
-                    <box size="${width} ${width} ${height3}"/>
-                </geometry>
-                <material name="orange"/>
-            </visual>
-            <inertial>
-                <origin xyz="0 0 ${height3/2 - axel_offset}" rpy="0 0 0"/>
-                <mass value="${mass}"/>
-                <inertia
-                        ixx="${mass / 12.0 * (width*width + height3*height3)}" ixy="0.0" ixz="0.0"
-                        iyy="${mass / 12.0 * (height3*height3 + width*width)}" iyz="0.0"
-                        izz="${mass / 12.0 * (width*width + width*width)}"/>
-            </inertial>
-        </link>
-        <joint name="${prefix}elbow_0_joint" type="revolute">
-            <parent link="${prefix}humerus_link"/>
-            <child link="${prefix}wrist_link"/>
-            <origin xyz="0 0 ${height3}" rpy="0 0 0"/>
-            <axis xyz="0 1 0"/>
-            <dynamics damping="0.7"/>
-            <limit lower="${-3*pi/4.0}" upper="${3*pi/4.0}" effort="100" velocity="1.0"/>
+        <!-- Joint from part_33 to flat_pattern_of_plate_1 -->
+        <joint name="elbow" type="revolute">
+            <origin xyz="0.4572 0.031582 -0.067374" rpy="-1.67319e-16 9.5285e-16 -3.14159"/>
+            <parent link="part_33"/>
+            <child link="flat_pattern_of_plate_1"/>
+            <axis xyz="0 0 1"/>
+            <limit effort="10" velocity="10" lower="-0.791612" upper="0.779185"/>
         </joint>
-        <!-- Wrist Link -->
-        <link name="${prefix}wrist_link">
-            <collision>
-                <origin xyz="0 0 ${height3/2 - axel_offset}" rpy="0 0 0"/>
-                <geometry>
-                    <box size="${width} ${width} ${height3}"/>
-                </geometry>
-            </collision>
-            <visual>
-                <origin xyz="0 0 ${height3/2 - axel_offset}" rpy="0 0 0"/>
-                <geometry>
-                    <box size="${width} ${width} ${height3}"/>
-                </geometry>
-                <material name="orange"/>
-            </visual>
-            <inertial>
-                <origin xyz="0 0 ${height3/2 - axel_offset}" rpy="0 0 0"/>
-                <mass value="${mass}"/>
-                <inertia
-                        ixx="${mass / 12.0 * (width*width + height3*height3)}" ixy="0.0" ixz="0.0"
-                        iyy="${mass / 12.0 * (height3*height3 + width*width)}" iyz="0.0"
-                        izz="${mass / 12.0 * (width*width + width*width)}"/>
-            </inertial>
-        </link>
-        <joint name="${prefix}gripper_wrist_fixture" type="fixed">
-            <parent link="${prefix}wrist_link"/>
-            <child link="${prefix}gripper_link"/>
-            <origin xyz="0 0 ${height3 - width}" rpy="0 0 0"/>
+        <!-- Joint from part_43 to part_33 -->
+        <joint name="base_pitch" type="revolute">
+            <origin xyz="-0.0204961 -1.85399e-16 -0.0851182" rpy="1.5708 1.44557 -1.5708"/>
+            <parent link="part_43"/>
+            <child link="part_33"/>
+            <axis xyz="0 0 1"/>
+            <limit effort="10" velocity="10" lower="-1.69602" upper="1.44557"/>
         </joint>
-        <!-- Gripper Link -->
-        <link name="${prefix}gripper_link">
-            <collision>
-                <origin xyz="0 0 ${gripper_thickness/2}" rpy="0 0 0"/>
-                <geometry>
-                    <box size="${gripper_width} ${gripper_breadth} ${gripper_thickness}"/>
-                </geometry>
-            </collision>
-            <visual>
-                <origin xyz="0 0 ${gripper_thickness/2}" rpy="0 0 0"/>
-                <geometry>
-                    <box size="${gripper_width} ${gripper_breadth} ${gripper_thickness}"/>
-                </geometry>
-                <material name="orange"/>
-            </visual>
-            <inertial>
-                <origin xyz="0 0 ${gripper_thickness/2}" rpy="0 0 0"/>
-                <mass value="${mass}"/>
-                <inertia
-                        ixx="${mass / 12.0 * (gripper_width*gripper_breadth + gripper_thickness*gripper_thickness)}" ixy="0.0" ixz="0.0"
-                        iyy="${mass / 12.0 * (gripper_thickness*gripper_thickness + gripper_width*gripper_breadth)}" iyz="0.0"
-                        izz="${mass / 12.0 * (gripper_width*gripper_breadth + gripper_width*gripper_breadth)}"/>
-            </inertial>
-        </link>
-        <joint name="${prefix}gripper" type="prismatic">
-            <origin xyz="${-gripper_width/2 - width/2} 0 ${gripper_thickness}" rpy="0 0 0"/>
-            <parent link="${prefix}gripper_link"/>
-            <child link="${prefix}finger_left_link"/>
-            <axis xyz="1 0 0"/>
-            <dynamics damping="0.7"/>
-            <limit lower="0" upper="${gripper_width/2 - finger_thickness}" effort="100" velocity="1.0"/>
+        <!-- Joint from part_48 to part_43 -->
+        <joint name="base_yaw" type="revolute">
+            <origin xyz="0.000390865 0.000967073 0.0809889" rpy="-3.1382 -0.0161184 -0.393065"/>
+            <parent link="part_48"/>
+            <child link="part_43"/>
+            <axis xyz="0 0 1"/>
+            <limit effort="10" velocity="10" lower="-3.141592653589793" upper="3.141592653589793"/>
         </joint>
-        <joint name="${prefix}gripper_mimic" type="prismatic">
-            <origin xyz="${-gripper_width/2 - width/2} 0 ${gripper_thickness}" rpy="0 0 0"/>
-            <parent link="${prefix}gripper_link"/>
-            <child link="${prefix}finger_right_link"/>
-            <mimic joint="${prefix}gripper" multiplier="-1" offset="0.5"/>
-            <axis xyz="1 0 0"/>
-            <dynamics damping="0.7"/>
-            <limit lower="${-gripper_width/2 + finger_thickness}" upper="0" effort="100" velocity="1.0"/>
-        </joint>
-        <!-- Finger Links -->
-        <link name="${prefix}finger_left_link">
-            <collision>
-                <origin xyz="${finger_thickness*1.5} 0 ${finger_length/2}" rpy="0 0 0"/>
-                <geometry>
-                    <box size="${finger_thickness} ${gripper_breadth} ${finger_length}"/>
-                </geometry>
-            </collision>
-            <visual>
-                <origin xyz="${finger_thickness*1.5} 0 ${finger_length/2}" rpy="0 0 0"/>
-                <geometry>
-                    <box size="${finger_thickness} ${gripper_breadth} ${finger_length}"/>
-                </geometry>
-                <material name="orange"/>
-            </visual>
-            <inertial>
-                <origin xyz="${finger_thickness*1.5} 0 ${finger_length/2}" rpy="0 0 0"/>
-                <mass value="${mass}"/>
-                <inertia
-                        ixx="${mass / 12.0 * (finger_thickness*gripper_breadth + finger_length*finger_length)}" ixy="0.0" ixz="0.0"
-                        iyy="${mass / 12.0 * (finger_length*finger_length + finger_thickness*gripper_breadth)}" iyz="0.0"
-                        izz="${mass / 12.0 * (finger_thickness*gripper_breadth + finger_thickness*gripper_breadth)}"/>
-            </inertial>
-        </link>
-        <link name="${prefix}finger_right_link">
-            <collision>
-                <origin xyz="${-finger_thickness*1.5} 0 ${finger_length/2}" rpy="0 0 0"/>
-                <geometry>
-                    <box size="${finger_thickness} ${width} ${finger_length}"/>
-                </geometry>
-            </collision>
-            <visual>
-                <origin xyz="${-finger_thickness*1.5} 0 ${finger_length/2}" rpy="0 0 0"/>
-                <geometry>
-                    <box size="${finger_thickness} ${width} ${finger_length}"/>
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