Commit message: Tweaked URDF

File: umrt-project-perry-description/urdf/project_perry_description.urdf.xacro (robot description, xacro)
@@ -2,12 +2,12 @@
 <robot xmlns:xacro="http://www.ros.org/wiki/xacro">
     <xacro:macro name="project_perry" params="parent prefix *origin">
-        <joint name="${prefix}base_joint" type="fixed">
+        <joint name="base_joint" type="fixed">
             <xacro:insert_block name="origin"/>
             <parent link="${parent}"/>
-            <child link="part_48"/>
+            <child link="base_link"/>
         </joint>
         <!-- Generated using onshape-to-robot -->
-        <!-- Link part_48 -->
-        <link name="part_48">
+        <!-- Link base_link -->
+        <link name="base_link">
             <inertial>
             <origin xyz="0.00286812 -0.0209097 0.0286943" rpy="0 0 0"/>
@@ -15,11 +15,11 @@
             <inertia ixx="0.0231691" ixy="0.00065571" ixz="-0.000230556" iyy="0.0147789" iyz="0.000656447" izz="0.0344912"/>
             </inertial>
-            <!-- Part part_48_parts -->
+            <!-- Part base_link_parts -->
             <visual>
             <origin xyz="0.00286812 -0.0209097 0.0286943" rpy="0 -0 0"/>
             <geometry>
-                <mesh filename="package://assets/merged/part_48_visual.stl"/>
+                <mesh filename="file://$(find umrt-project-perry-description)/assets/merged/part_48_visual.stl"/>
             </geometry>
-            <material name="part_48_parts_material">
+            <material name="base_link_parts_material">
                 <color rgba="0.0745098 0.678431 0.972549 1"/>
             </material>
@@ -28,5 +28,5 @@
             <origin xyz="0.00286812 -0.0209097 0.0286943" rpy="0 -0 0"/>
             <geometry>
-                <mesh filename="package://assets/merged/part_48_collision.stl"/>
+                <mesh filename="file://$(find umrt-project-perry-description)/assets/merged/part_48_collision.stl"/>
             </geometry>
             </collision>
@@ -43,5 +43,5 @@
             <origin xyz="-0.0119595 -0.00118557 -0.0231327" rpy="-3.13855 -0.016189 -0.393062"/>
             <geometry>
-                <mesh filename="package://assets/merged/part_43_visual.stl"/>
+                <mesh filename="file://$(find umrt-project-perry-description)/assets/merged/part_43_visual.stl"/>
             </geometry>
             <material name="part_43_parts_material">
@@ -52,5 +52,5 @@
             <origin xyz="-0.0119595 -0.00118557 -0.0231327" rpy="-3.13855 -0.016189 -0.393062"/>
             <geometry>
-                <mesh filename="package://assets/merged/part_43_collision.stl"/>
+                <mesh filename="file://$(find umrt-project-perry-description)/assets/merged/part_43_collision.stl"/>
             </geometry>
             </collision>
@@ -67,5 +67,5 @@
             <origin xyz="0.191821 -0.0003306 -0.0214358" rpy="1.61286 1.17742 1.48782"/>
             <geometry>
-                <mesh filename="package://assets/merged/part_33_visual.stl"/>
+                <mesh filename="file://$(find umrt-project-perry-description)/assets/merged/part_33_visual.stl"/>
             </geometry>
             <material name="part_33_parts_material">
@@ -76,5 +76,5 @@
             <origin xyz="0.191821 -0.0003306 -0.0214358" rpy="1.61286 1.17742 1.48782"/>
             <geometry>
-                <mesh filename="package://assets/merged/part_33_collision.stl"/>
+                <mesh filename="file://$(find umrt-project-perry-description)/assets/merged/part_33_collision.stl"/>
             </geometry>
             </collision>
@@ -91,5 +91,5 @@
             <origin xyz="0.0157793 -0.119702 0.0450796" rpy="1.61286 1.17742 -1.65378"/>
             <geometry>
-                <mesh filename="package://assets/merged/flat_pattern_of_plate_1_visual.stl"/>
+                <mesh filename="file://$(find umrt-project-perry-description)/assets/merged/flat_pattern_of_plate_1_visual.stl"/>
             </geometry>
             <material name="flat_pattern_of_plate_1_parts_material">
@@ -100,5 +100,5 @@
             <origin xyz="0.0157793 -0.119702 0.0450796" rpy="1.61286 1.17742 -1.65378"/>
             <geometry>
-                <mesh filename="package://assets/merged/flat_pattern_of_plate_1_collision.stl"/>
+                <mesh filename="file://$(find umrt-project-perry-description)/assets/merged/flat_pattern_of_plate_1_collision.stl"/>
             </geometry>
             </collision>
@@ -115,5 +115,5 @@
             <origin xyz="1.74216e-05 -0.0133229 -0.0449775" rpy="1.61286 1.17742 -1.4845"/>
             <geometry>
-                <mesh filename="package://assets/merged/part_6_visual.stl"/>
+                <mesh filename="file://$(find umrt-project-perry-description)/assets/merged/part_6_visual.stl"/>
             </geometry>
             <material name="part_6_parts_material">
@@ -124,5 +124,5 @@
             <origin xyz="1.74216e-05 -0.0133229 -0.0449775" rpy="1.61286 1.17742 -1.4845"/>
             <geometry>
-                <mesh filename="package://assets/merged/part_6_collision.stl"/>
+                <mesh filename="file://$(find umrt-project-perry-description)/assets/merged/part_6_collision.stl"/>
             </geometry>
             </collision>
@@ -139,5 +139,5 @@
             <origin xyz="-2.77556e-17 5.55112e-17 -0.00183593" rpy="-1.62212 0.391834 -2.8036"/>
             <geometry>
-                <mesh filename="package://assets/merged/part_8_visual.stl"/>
+                <mesh filename="file://$(find umrt-project-perry-description)/assets/merged/part_8_visual.stl"/>
             </geometry>
             <material name="part_8_parts_material">
@@ -148,5 +148,5 @@
             <origin xyz="-2.77556e-17 5.55112e-17 -0.00183593" rpy="-1.62212 0.391834 -2.8036"/>
             <geometry>
-                <mesh filename="package://assets/merged/part_8_collision.stl"/>
+                <mesh filename="file://$(find umrt-project-perry-description)/assets/merged/part_8_collision.stl"/>
             </geometry>
             </collision>
@@ -169,5 +169,5 @@
         </joint>
         <!-- Joint from part_33 to flat_pattern_of_plate_1 -->
-        <joint name="elbow" type="revolute">
+        <joint name="elbow_0_joint" type="revolute">
             <origin xyz="0.4572 0.031582 -0.067374" rpy="-1.67319e-16 9.5285e-16 -3.14159"/>
             <parent link="part_33"/>
@@ -184,8 +184,8 @@
             <limit effort="10" velocity="10" lower="-1.69602" upper="1.44557"/>
         </joint>
-        <!-- Joint from part_48 to part_43 -->
+        <!-- Joint from base_link to part_43 -->
         <joint name="base_yaw" type="revolute">
             <origin xyz="0.000390865 0.000967073 0.0809889" rpy="-3.1382 -0.0161184 -0.393065"/>
-            <parent link="part_48"/>
+            <parent link="base_link"/>
             <child link="part_43"/>
             <axis xyz="0 0 1"/>
