Commit message: Re-applied URDF tweaks

File: umrt-project-perry-description/urdf/project_perry_description.urdf.xacro (robot description, xacro)
@@ -19,5 +19,5 @@
                 <origin xyz="0.00286812 -0.0209097 0.0286943" rpy="0 -0 0"/>
                 <geometry>
-                    <mesh filename="package://assets/merged/base_link_visual.stl"/>
+                    <mesh filename="file://$(find umrt-project-perry-description)/assets/merged/base_link_visual.stl"/>
                 </geometry>
                 <material name="base_link_parts_material">
@@ -28,5 +28,5 @@
                 <origin xyz="0.00286812 -0.0209097 0.0286943" rpy="0 -0 0"/>
                 <geometry>
-                    <mesh filename="package://assets/merged/base_link_collision.stl"/>
+                    <mesh filename="file://$(find umrt-project-perry-description)/assets/merged/base_link_collision.stl"/>
                 </geometry>
             </collision>
@@ -43,5 +43,5 @@
                 <origin xyz="-0.0119595 -0.00118557 -0.0231327" rpy="-3.13855 -0.016189 0.947366"/>
                 <geometry>
-                    <mesh filename="package://assets/merged/base_platter_visual.stl"/>
+                    <mesh filename="file://$(find umrt-project-perry-description)/assets/merged/base_platter_visual.stl"/>
                 </geometry>
                 <material name="base_platter_parts_material">
@@ -52,5 +52,5 @@
                 <origin xyz="-0.0119595 -0.00118557 -0.0231327" rpy="-3.13855 -0.016189 0.947366"/>
                 <geometry>
-                    <mesh filename="package://assets/merged/base_platter_collision.stl"/>
+                    <mesh filename="file://$(find umrt-project-perry-description)/assets/merged/base_platter_collision.stl"/>
                 </geometry>
             </collision>
@@ -67,5 +67,5 @@
                 <origin xyz="0.192899 1.61439e-05 -0.0214358" rpy="-1.5794 0.623336 -1.23434"/>
                 <geometry>
-                    <mesh filename="package://assets/merged/humerus_link_visual.stl"/>
+                    <mesh filename="file://$(find umrt-project-perry-description)/assets/merged/humerus_link_visual.stl"/>
                 </geometry>
                 <material name="humerus_link_parts_material">
@@ -76,5 +76,5 @@
                 <origin xyz="0.192899 1.61439e-05 -0.0214358" rpy="-1.5794 0.623336 -1.23434"/>
                 <geometry>
-                    <mesh filename="package://assets/merged/humerus_link_collision.stl"/>
+                    <mesh filename="file://$(find umrt-project-perry-description)/assets/merged/humerus_link_collision.stl"/>
                 </geometry>
             </collision>
@@ -91,5 +91,5 @@
                 <origin xyz="0.0461837 -0.111635 0.0450797" rpy="-1.5794 0.623336 1.90726"/>
                 <geometry>
-                    <mesh filename="package://assets/merged/flat_pattern_of_humerus_link_visual.stl"/>
+                    <mesh filename="file://$(find umrt-project-perry-description)/assets/merged/flat_pattern_of_humerus_link_visual.stl"/>
                 </geometry>
                 <material name="flat_pattern_of_humerus_link_parts_material">
@@ -100,5 +100,5 @@
                 <origin xyz="0.0461837 -0.111635 0.0450797" rpy="-1.5794 0.623336 1.90726"/>
                 <geometry>
-                    <mesh filename="package://assets/merged/flat_pattern_of_humerus_link_collision.stl"/>
+                    <mesh filename="file://$(find umrt-project-perry-description)/assets/merged/flat_pattern_of_humerus_link_collision.stl"/>
                 </geometry>
             </collision>
@@ -115,5 +115,5 @@
                 <origin xyz="1.74216e-05 -0.0133229 -0.0449775" rpy="-1.5794 0.623336 1.87508"/>
                 <geometry>
-                    <mesh filename="package://assets/merged/wirst_body_visual.stl"/>
+                    <mesh filename="file://$(find umrt-project-perry-description)/assets/merged/wirst_body_visual.stl"/>
                 </geometry>
                 <material name="wirst_body_parts_material">
@@ -124,5 +124,5 @@
                 <origin xyz="1.74216e-05 -0.0133229 -0.0449775" rpy="-1.5794 0.623336 1.87508"/>
                 <geometry>
-                    <mesh filename="package://assets/merged/wirst_body_collision.stl"/>
+                    <mesh filename="file://$(find umrt-project-perry-description)/assets/merged/wirst_body_collision.stl"/>
                 </geometry>
             </collision>
@@ -139,5 +139,5 @@
                 <origin xyz="0 6.93889e-18 -0.00183593" rpy="-2.07296 -0.886139 2.06643"/>
                 <geometry>
-                    <mesh filename="package://assets/merged/wrist_link_visual.stl"/>
+                    <mesh filename="file://$(find umrt-project-perry-description)/assets/merged/wrist_link_visual.stl"/>
                 </geometry>
                 <material name="wrist_link_parts_material">
@@ -148,5 +148,5 @@
                 <origin xyz="0 6.93889e-18 -0.00183593" rpy="-2.07296 -0.886139 2.06643"/>
                 <geometry>
-                    <mesh filename="package://assets/merged/wrist_link_collision.stl"/>
+                    <mesh filename="file://$(find umrt-project-perry-description)/assets/merged/wrist_link_collision.stl"/>
                 </geometry>
             </collision>

Commit message: Updated model again

File: umrt-project-perry-description/urdf/project_perry_description.urdf.xacro (robot description, xacro)
@@ -19,5 +19,5 @@
                 <origin xyz="0.00286812 -0.0209097 0.0286943" rpy="0 -0 0"/>
                 <geometry>
-                    <mesh filename="file://$(find umrt-project-perry-description)/assets/merged/base_link_visual.stl"/>
+                    <mesh filename="package://assets/merged/base_link_visual.stl"/>
                 </geometry>
                 <material name="base_link_parts_material">
@@ -28,5 +28,5 @@
                 <origin xyz="0.00286812 -0.0209097 0.0286943" rpy="0 -0 0"/>
                 <geometry>
-                    <mesh filename="file://$(find umrt-project-perry-description)/assets/merged/base_link_collision.stl"/>
+                    <mesh filename="package://assets/merged/base_link_collision.stl"/>
                 </geometry>
             </collision>
@@ -41,7 +41,7 @@
             <!-- Part base_platter_parts -->
             <visual>
-                <origin xyz="-0.0119595 -0.00118557 -0.0231327" rpy="-3.13855 -0.016189 0.947366"/>
-                <geometry>
-                    <mesh filename="file://$(find umrt-project-perry-description)/assets/merged/base_platter_visual.stl"/>
+                <origin xyz="-0.0119595 -0.00118557 -0.0231327" rpy="-3.13855 -0.016189 0.0123501"/>
+                <geometry>
+                    <mesh filename="package://assets/merged/base_platter_visual.stl"/>
                 </geometry>
                 <material name="base_platter_parts_material">
@@ -50,7 +50,7 @@
             </visual>
             <collision>
-                <origin xyz="-0.0119595 -0.00118557 -0.0231327" rpy="-3.13855 -0.016189 0.947366"/>
-                <geometry>
-                    <mesh filename="file://$(find umrt-project-perry-description)/assets/merged/base_platter_collision.stl"/>
+                <origin xyz="-0.0119595 -0.00118557 -0.0231327" rpy="-3.13855 -0.016189 0.0123501"/>
+                <geometry>
+                    <mesh filename="package://assets/merged/base_platter_collision.stl"/>
                 </geometry>
             </collision>
@@ -59,13 +59,13 @@
         <link name="humerus_link">
             <inertial>
-                <origin xyz="0.192899 1.61439e-05 -0.0214358" rpy="0 0 0"/>
+                <origin xyz="0.19104 -0.000401365 -0.0214358" rpy="0 0 0"/>
                 <mass value="2.10608"/>
-                <inertia ixx="0.00597093" ixy="-0.00115128" ixz="-0.000267892" iyy="0.0356475" iyz="-2.43475e-05" izz="0.0374601"/>
+                <inertia ixx="0.00612771" ixy="-0.00148492" ixz="-0.000269689" iyy="0.0355118" iyz="-2.47513e-05" izz="0.0374813"/>
             </inertial>
             <!-- Part humerus_link_parts -->
             <visual>
-                <origin xyz="0.192899 1.61439e-05 -0.0214358" rpy="-1.5794 0.623336 -1.23434"/>
-                <geometry>
-                    <mesh filename="file://$(find umrt-project-perry-description)/assets/merged/humerus_link_visual.stl"/>
+                <origin xyz="0.19104 -0.000401365 -0.0214358" rpy="-2.48682 1.55043 -2.48996"/>
+                <geometry>
+                    <mesh filename="package://assets/merged/humerus_link_visual.stl"/>
                 </geometry>
                 <material name="humerus_link_parts_material">
@@ -74,7 +74,7 @@
             </visual>
             <collision>
-                <origin xyz="0.192899 1.61439e-05 -0.0214358" rpy="-1.5794 0.623336 -1.23434"/>
-                <geometry>
-                    <mesh filename="file://$(find umrt-project-perry-description)/assets/merged/humerus_link_collision.stl"/>
+                <origin xyz="0.19104 -0.000401365 -0.0214358" rpy="-2.48682 1.55043 -2.48996"/>
+                <geometry>
+                    <mesh filename="package://assets/merged/humerus_link_collision.stl"/>
                 </geometry>
             </collision>
@@ -83,13 +83,13 @@
         <link name="flat_pattern_of_humerus_link">
             <inertial>
-                <origin xyz="0.0461837 -0.111635 0.0450797" rpy="0 0 0"/>
+                <origin xyz="-0.00600861 -0.120661 0.0450797" rpy="0 0 0"/>
                 <mass value="2.41904"/>
-                <inertia ixx="0.0549307" ixy="0.0238789" ixz="-1.1312e-05" iyy="0.0212463" iyz="1.93753e-05" izz="0.064383"/>
+                <inertia ixx="0.0672327" ixy="0.0021158" ixz="-1.93671e-06" iyy="0.00894428" iyz="2.2352e-05" izz="0.064383"/>
             </inertial>
             <!-- Part flat_pattern_of_humerus_link_parts -->
             <visual>
-                <origin xyz="0.0461837 -0.111635 0.0450797" rpy="-1.5794 0.623336 1.90726"/>
-                <geometry>
-                    <mesh filename="file://$(find umrt-project-perry-description)/assets/merged/flat_pattern_of_humerus_link_visual.stl"/>
+                <origin xyz="-0.00600861 -0.120661 0.0450797" rpy="-2.48682 1.55043 0.651633"/>
+                <geometry>
+                    <mesh filename="package://assets/merged/flat_pattern_of_humerus_link_visual.stl"/>
                 </geometry>
                 <material name="flat_pattern_of_humerus_link_parts_material">
@@ -98,7 +98,7 @@
             </visual>
             <collision>
-                <origin xyz="0.0461837 -0.111635 0.0450797" rpy="-1.5794 0.623336 1.90726"/>
-                <geometry>
-                    <mesh filename="file://$(find umrt-project-perry-description)/assets/merged/flat_pattern_of_humerus_link_collision.stl"/>
+                <origin xyz="-0.00600861 -0.120661 0.0450797" rpy="-2.48682 1.55043 0.651633"/>
+                <geometry>
+                    <mesh filename="package://assets/merged/flat_pattern_of_humerus_link_collision.stl"/>
                 </geometry>
             </collision>
@@ -113,7 +113,7 @@
             <!-- Part wirst_body_parts -->
             <visual>
-                <origin xyz="1.74216e-05 -0.0133229 -0.0449775" rpy="-1.5794 0.623336 1.87508"/>
-                <geometry>
-                    <mesh filename="file://$(find umrt-project-perry-description)/assets/merged/wirst_body_visual.stl"/>
+                <origin xyz="1.74216e-05 -0.0133229 -0.0449775" rpy="-2.48682 1.55043 0.651633"/>
+                <geometry>
+                    <mesh filename="package://assets/merged/wirst_body_visual.stl"/>
                 </geometry>
                 <material name="wirst_body_parts_material">
@@ -122,7 +122,7 @@
             </visual>
             <collision>
-                <origin xyz="1.74216e-05 -0.0133229 -0.0449775" rpy="-1.5794 0.623336 1.87508"/>
-                <geometry>
-                    <mesh filename="file://$(find umrt-project-perry-description)/assets/merged/wirst_body_collision.stl"/>
+                <origin xyz="1.74216e-05 -0.0133229 -0.0449775" rpy="-2.48682 1.55043 0.651633"/>
+                <geometry>
+                    <mesh filename="package://assets/merged/wirst_body_collision.stl"/>
                 </geometry>
             </collision>
@@ -131,13 +131,13 @@
         <link name="wrist_link">
             <inertial>
-                <origin xyz="-1.636e-17 -6.74869e-18 -0.00183593" rpy="0 0 0"/>
+                <origin xyz="-2.16903e-18 -4.83311e-17 -0.00183593" rpy="0 0 0"/>
                 <mass value="0.0230672"/>
-                <inertia ixx="6.54736e-06" ixy="1.482e-22" ixz="1.20262e-21" iyy="6.54736e-06" iyz="-9.13762e-22" izz="1.27521e-05"/>
+                <inertia ixx="6.54736e-06" ixy="-2.51728e-23" ixz="-4.00656e-23" iyy="6.54736e-06" iyz="-5.94725e-24" izz="1.27521e-05"/>
             </inertial>
             <!-- Part wrist_link_parts -->
             <visual>
-                <origin xyz="0 6.93889e-18 -0.00183593" rpy="-2.07296 -0.886139 2.06643"/>
-                <geometry>
-                    <mesh filename="file://$(find umrt-project-perry-description)/assets/merged/wrist_link_visual.stl"/>
+                <origin xyz="-2.1684e-18 0 -0.00183593" rpy="-1.56756 -0.0123485 -0.0161902"/>
+                <geometry>
+                    <mesh filename="package://assets/merged/wrist_link_visual.stl"/>
                 </geometry>
                 <material name="wrist_link_parts_material">
@@ -146,13 +146,28 @@
             </visual>
             <collision>
-                <origin xyz="0 6.93889e-18 -0.00183593" rpy="-2.07296 -0.886139 2.06643"/>
-                <geometry>
-                    <mesh filename="file://$(find umrt-project-perry-description)/assets/merged/wrist_link_collision.stl"/>
-                </geometry>
-            </collision>
-        </link>
+                <origin xyz="-2.1684e-18 0 -0.00183593" rpy="-1.56756 -0.0123485 -0.0161902"/>
+                <geometry>
+                    <mesh filename="package://assets/merged/wrist_link_collision.stl"/>
+                </geometry>
+            </collision>
+        </link>
+        <!-- Frame toolpoint (dummy link + fixed joint) -->
+        <link name="toolpoint">
+            <origin xyz="0 0 0" rpy="0 -0 0"/>
+            <inertial>
+                <origin xyz="0 0 0" rpy="0 0 0"/>
+                <mass value="1e-9"/>
+                <inertia ixx="0" ixy="0" ixz="0" iyy="0" iyz="0" izz="0"/>
+            </inertial>
+        </link>
+        <joint name="toolpoint_frame" type="fixed">
+            <origin xyz="6.01645e-15 -3.66374e-14 -0.185923" rpy="-2.31486e-13 -2.82334e-14 2.83915e-14"/>
+            <parent link="wrist_link"/>
+            <child link="toolpoint"/>
+            <axis xyz="0 0 0"/>
+        </joint>
         <!-- Joint from wirst_body to wrist_link -->
         <joint name="wrist_roll" type="revolute">
-            <origin xyz="-5.55112e-17 -0.0314483 -0.0449775" rpy="-1.5708 -0.100784 4.27299e-14"/>
+            <origin xyz="2.22045e-16 -0.0314483 -0.0449775" rpy="-1.5708 1.5708 0"/>
             <parent link="wirst_body"/>
             <child link="wrist_link"/>
@@ -162,29 +177,29 @@
         <!-- Joint from flat_pattern_of_humerus_link to wirst_body -->
         <joint name="wrist_pitch" type="revolute">
-            <origin xyz="0.168411 -0.355861 0.0899558" rpy="5.38276e-15 -3.06298e-16 0.0321741"/>
+            <origin xyz="1.77636e-15 -0.3937 0.0899558" rpy="1.67261e-15 -2.51166e-15 -1.23947e-15"/>
             <parent link="flat_pattern_of_humerus_link"/>
             <child link="wirst_body"/>
             <axis xyz="0 0 1"/>
-            <limit effort="10" velocity="10" lower="-1.16095" upper="1.98064"/>
+            <limit effort="10" velocity="10" lower="-1.5708" upper="1.5708"/>
         </joint>
         <!-- Joint from humerus_link to flat_pattern_of_humerus_link -->
         <joint name="elbow_pitch" type="revolute">
-            <origin xyz="0.4572 0.031582 -0.067374" rpy="-7.74298e-17 1.17778e-15 -3.14159"/>
+            <origin xyz="0.4572 0.031582 -0.067374" rpy="5.83832e-15 6.48493e-15 -3.14159"/>
             <parent link="humerus_link"/>
             <child link="flat_pattern_of_humerus_link"/>
             <axis xyz="0 0 1"/>
-            <limit effort="10" velocity="10" lower="-1.05288" upper="0.517911"/>
+            <limit effort="10" velocity="10" lower="-0.610865" upper="0.959931"/>
         </joint>
         <!-- Joint from base_platter to humerus_link -->
         <joint name="base_pitch" type="revolute">
-            <origin xyz="-0.0204961 7.17742e-17 -0.0851182" rpy="-1.5708 1.2144 1.5708"/>
+            <origin xyz="-0.0204961 -7.37257e-18 -0.0851182" rpy="-3.14159 1.5708 0"/>
             <parent link="base_platter"/>
             <child link="humerus_link"/>
             <axis xyz="0 0 1"/>
-            <limit effort="10" velocity="10" lower="-1.2144" upper="1.9272"/>
+            <limit effort="10" velocity="10" lower="-1.5708" upper="1.5708"/>
         </joint>
         <!-- Joint from base_link to base_platter -->
         <joint name="base_yaw" type="revolute">
-            <origin xyz="0.000390865 0.000967073 0.0809889" rpy="3.12667 -0.00698374 0.947443"/>
+            <origin xyz="0.000390865 0.000967073 0.0809889" rpy="3.13835 -0.0161502 0.0124009"/>
             <parent link="base_link"/>
             <child link="base_platter"/>

File: umrt-project-perry-description/urdf/robot.urdf (robot description, URDF)
Before this commit: robot pp-arm3, 6 links, 5 joints
Links:
- added link toolpoint, mass 1e-9
Joints:
- added joint toolpoint_frame: type fixed, parent wrist_link, child toolpoint, origin xyz=6.01645e-15 -3.66374e-14 -0.185923 rpy=-2.31486e-13 -2.82334e-14 2.83915e-14, axis 0 0 0
- joint base_pitch: limit lower=-1.2144 upper=1.9272 effort=10 velocity=10 -> lower=-1.5708 upper=1.5708 effort=10 velocity=10; origin xyz=-0.0204961 7.17742e-17 -0.0851182 rpy=-1.5708 1.2144 1.5708 -> xyz=-0.0204961 -7.37257e-18 -0.0851182 rpy=-3.14159 1.5708 0
- joint base_yaw: origin xyz=0.000390865 0.000967073 0.0809889 rpy=3.12667 -0.00698374 0.947443 -> xyz=0.000390865 0.000967073 0.0809889 rpy=3.13835 -0.0161502 0.0124009
- joint elbow_pitch: limit lower=-1.05288 upper=0.517911 effort=10 velocity=10 -> lower=-0.610865 upper=0.959931 effort=10 velocity=10; origin xyz=0.4572 0.031582 -0.067374 rpy=-7.74298e-17 1.17778e-15 -3.14159 -> xyz=0.4572 0.031582 -0.067374 rpy=5.83832e-15 6.48493e-15 -3.14159
- joint wrist_pitch: limit lower=-1.16095 upper=1.98064 effort=10 velocity=10 -> lower=-1.5708 upper=1.5708 effort=10 velocity=10; origin xyz=0.168411 -0.355861 0.0899558 rpy=5.38276e-15 -3.06298e-16 0.0321741 -> xyz=1.77636e-15 -0.3937 0.0899558 rpy=1.67261e-15 -2.51166e-15 -1.23947e-15
- joint wrist_roll: origin xyz=-5.55112e-17 -0.0314483 -0.0449775 rpy=-1.5708 -0.100784 4.27299e-14 -> xyz=2.22045e-16 -0.0314483 -0.0449775 rpy=-1.5708 1.5708 0
