Commit message: Added fake gripper link+joint to shut up some error messages when gripper GPIO is added

File: umrt-project-perry-description/urdf/project_perry_description.urdf.xacro (robot description, xacro)
@@ -152,4 +152,26 @@
             </collision>
         </link>
+        <link name="gripper_finger">
+            <inertial>
+                <origin xyz="0 0 0" rpy="0 0 0"/>
+                <mass value="0.0"/>
+                <inertia ixx="0.0" ixy="0.0" ixz="0.0" iyy="0.0" iyz="0.0" izz="0.0"/>
+            </inertial>
+            <!-- Part gripper_interface -->
+            <visual>
+                <origin xyz="0 0 0" rpy="0 0 0"/>
+                <material name="gripper_interface_material">
+                    <color rgba="0.498039 0.498039 0.498039 1"/>
+                </material>
+            </visual>
+            <collision>
+                <origin xyz="0 0 0" rpy="0 0 0"/>
+            </collision>
+        </link>
+        <joint name="gripper" type="fixed">
+            <origin xyz="0 0 0" rpy="0 0 0"/>
+            <parent link="gripper_interface"/>
+            <child link="gripper_finger"/>
+        </joint>
         <!-- Joint from wrist_link to gripper_interface -->
         <joint name="wrist_roll" type="revolute">
