Commit message: Update joint limits for robotic arm

File: umrt-project-perry-description/urdf/project_perry_description.urdf.xacro (robot description, xacro)
@@ -196,5 +196,6 @@
             <child link="ulna_link"/>
             <axis xyz="0 0 1"/>
-            <limit effort="10" velocity="10" lower="-0.959931" upper="0.610865"/>
+            <!-- 40 degrees back, 40 degrees forward -->
+            <limit effort="10" velocity="10" lower="-0.6981317" upper="0.6981317"/>
         </joint>
         <!-- Joint from platter_link to humerus_link -->
@@ -204,5 +205,6 @@
             <child link="humerus_link"/>
             <axis xyz="0 0 1"/>
-            <limit effort="10" velocity="10" lower="-1.5708" upper="1.5708"/>
+            <!-- 30 degrees back, 70 degrees forward -->
+            <limit effort="10" velocity="10" lower="-0.5235" upper="1.22173"/>
         </joint>
         <!-- Joint from base_link to platter_link -->
@@ -212,5 +214,6 @@
             <child link="platter_link"/>
             <axis xyz="0 0 1"/>
-            <limit effort="10" velocity="10" lower="-3.141592653589793" upper="3.141592653589793"/>
+            <!-- 3 pi each way ==> three revolutions -->
+            <limit effort="10" velocity="10" lower="-9.42" upper="9.42"/>
         </joint>
     </xacro:macro>

Commit message: Invert certain robotic arm axes.
This is a temporary fix for an underlying issue with the robotic arm
in umrt-arm-ros-firmware.

We need to add a configuration option to invert the requested angle coming from the ros controller.

File: umrt-project-perry-description/urdf/project_perry_description.urdf.xacro (robot description, xacro)
@@ -195,5 +195,5 @@
             <parent link="humerus_link"/>
             <child link="ulna_link"/>
-            <axis xyz="0 0 1"/>
+            <axis xyz="0 0 -1"/>
             <!-- 40 degrees back, 40 degrees forward -->
             <limit effort="10" velocity="10" lower="-0.6981317" upper="0.6981317"/>
@@ -204,7 +204,7 @@
             <parent link="platter_link"/>
             <child link="humerus_link"/>
-            <axis xyz="0 0 1"/>
+            <axis xyz="0 0 -1"/>
             <!-- 30 degrees back, 70 degrees forward -->
-            <limit effort="10" velocity="10" lower="-0.5235" upper="1.22173"/>
+            <limit effort="10" velocity="10" lower="-1.22173" upper="0.5235"/>
         </joint>
         <!-- Joint from base_link to platter_link -->
@@ -215,5 +215,5 @@
             <axis xyz="0 0 1"/>
             <!-- 3 pi each way ==> three revolutions -->
-            <limit effort="10" velocity="10" lower="-9.42" upper="9.42"/>
+            <limit effort="10" velocity="10" lower="-3.14" upper="3.14"/>
         </joint>
     </xacro:macro>
