Commit message: Rolled back model IKFast works

File: ik2/project_perry_description.urdf.xacro (robot description, xacro)
@@ -7,204 +7,236 @@
             <child link="base_link"/>
         </joint>
+        <!-- Constants for robot dimensions -->
+        <xacro:property name="mass" value="1"/> <!-- arbitrary value for mass -->
+        <xacro:property name="base_width" value="1"/>
+        <xacro:property name="base_height" value="0.6"/>
+        <xacro:property name="platter_radius" value="0.75"/>
+        <xacro:property name="platter_height" value="0.1"/>
+        <xacro:property name="width" value="0.1"/> <!-- Square dimensions (widthxwidth) of beams -->
+        <xacro:property name="height1" value="2"/> <!-- Link 1 -->
+        <xacro:property name="height2" value="1"/> <!-- Link 2 -->
+        <xacro:property name="height3" value="1"/> <!-- Link 3 -->
+        <xacro:property name="gripper_width" value="0.4"/>
+        <xacro:property name="gripper_breadth" value="0.1"/>
+        <xacro:property name="gripper_thickness" value="0.05"/>
+        <xacro:property name="finger_length" value="0.2"/>
+        <xacro:property name="finger_thickness" value="0.05"/>
+        <xacro:property name="axel_offset" value="0.05"/> <!-- Space btw top of beam and the each joint -->
         <!-- Generated using onshape-to-robot -->
-        <!-- Link base_link -->
+        <!-- Base Link -->
         <link name="base_link">
-            <inertial>
-                <origin xyz="0.00286812 -0.0209097 0.0286943" rpy="0 0 0"/>
-                <mass value="2.80632"/>
-                <inertia ixx="0.0231691" ixy="0.00065571" ixz="-0.000230556" iyy="0.0147789" iyz="0.000656447" izz="0.0344912"/>
-            </inertial>
-            <!-- Part base_link_parts -->
-            <visual>
-                <origin xyz="0.00286812 -0.0209097 0.0286943" rpy="0 -0 0"/>
-                <geometry>
-                    <mesh filename="file://$(find umrt-project-perry-description)/assets/merged/base_link_visual.stl"/>
-                </geometry>
-                <material name="base_link_parts_material">
-                    <color rgba="0.0745098 0.678431 0.972549 1"/>
-                </material>
-            </visual>
-            <collision>
-                <origin xyz="0.00286812 -0.0209097 0.0286943" rpy="0 -0 0"/>
-                <geometry>
-                    <mesh filename="file://$(find umrt-project-perry-description)/assets/merged/base_link_collision.stl"/>
-                </geometry>
-            </collision>
-        </link>
-        <!-- Link base_platter -->
-        <link name="base_platter">
-            <inertial>
-                <origin xyz="-0.0119595 -0.00118557 -0.0231327" rpy="0 0 0"/>
-                <mass value="1.84265"/>
-                <inertia ixx="0.00590316" ixy="0.000138602" ixz="-0.000532603" iyy="0.00955076" iyz="2.11489e-05" izz="0.012905"/>
-            </inertial>
-            <!-- Part base_platter_parts -->
-            <visual>
-                <origin xyz="-0.0119595 -0.00118557 -0.0231327" rpy="-3.13855 -0.016189 0.0123501"/>
-                <geometry>
-                    <mesh filename="file://$(find umrt-project-perry-description)/assets/merged/base_platter_visual.stl"/>
-                </geometry>
-                <material name="base_platter_parts_material">
-                    <color rgba="0.570634 0.573152 0.433741 1"/>
-                </material>
-            </visual>
-            <collision>
-                <origin xyz="-0.0119595 -0.00118557 -0.0231327" rpy="-3.13855 -0.016189 0.0123501"/>
-                <geometry>
-                    <mesh filename="file://$(find umrt-project-perry-description)/assets/merged/base_platter_collision.stl"/>
-                </geometry>
-            </collision>
-        </link>
-        <!-- Link humerus_link -->
+            <collision>
+                <origin xyz="0 0 ${base_height/2}" rpy="0 0 0"/>
+                <geometry>
+                    <box size="${base_width} ${base_width} ${base_height}"/>
+                </geometry>
+            </collision>
+            <visual>
+                <origin xyz="0 0 ${base_height/2}" rpy="0 0 0"/>
+                <geometry>
+                    <box size="${base_width} ${base_width} ${base_height}"/>
+                </geometry>
+                <material name="orange"/>
+            </visual>
+            <inertial>
+                <origin xyz="0 0 ${base_height/2}" rpy="0 0 0"/>
+                <mass value="${mass}"/>
+                <inertia
+                        ixx="${mass / 12.0 * (base_width*base_width + base_height*base_height)}" ixy="0.0" ixz="0.0"
+                        iyy="${mass / 12.0 * (base_height*base_height + base_width*base_width)}" iyz="0.0"
+                        izz="${mass / 12.0 * (base_width*base_width + base_width*base_width)}"/>
+            </inertial>
+        </link>
+        <joint name="base_yaw_joint" type="continuous">
+            <parent link="base_link"/>
+            <child link="shoulder_link"/>
+            <origin xyz="0 0 ${base_height - axel_offset}" rpy="0 0 0"/>
+            <axis xyz="0 0 1"/>
+            <dynamics damping="0.7"/>
+            <limit effort="100" velocity="1.0"/>
+        </joint>
+        <!-- Middle Link -->
+        <link name="shoulder_link">
+            <collision>
+                <origin xyz="0 0 ${platter_height/2 + axel_offset}" rpy="0 0 0"/>
+                <geometry>
+                    <cylinder radius="${platter_radius}" length="${platter_height}"/>
+                </geometry>
+            </collision>
+            <visual>
+                <origin xyz="0 0 ${platter_height/2 + axel_offset}" rpy="0 0 0"/>
+                <geometry>
+                    <cylinder radius="${platter_radius}" length="${platter_height}"/>
+                </geometry>
+                <material name="yellow"/>
+            </visual>
+            <inertial>
+                <origin xyz="0 0 ${platter_height/2 - axel_offset}" rpy="0 0 0"/>
+                <mass value="${mass}"/>
+                <inertia
+                        ixx="${mass / 12.0 * (3*platter_radius*platter_radius + platter_height*platter_height)}"
+                        ixy="0.0" ixz="0.0"
+                        iyy="${mass / 12.0 * (3*platter_radius*platter_radius + platter_height*platter_height)}"
+                        iyz="0.0"
+                        izz="${mass / 2.0 * platter_radius*platter_radius}"/>
+            </inertial>
+        </link>
+        <joint name="base_pitch_joint" type="revolute">
+            <parent link="shoulder_link"/>
+            <child link="humerus_link"/>
+            <origin xyz="0 0 ${platter_height + axel_offset*2}" rpy="0 0 0"/>
+            <axis xyz="0 1 0"/>
+            <dynamics damping="0.7"/>
+            <limit lower="${-pi/2.0}" upper="${pi/2.0}" effort="100" velocity="1.0"/>
+        </joint>
+        <!-- Top Link -->
         <link name="humerus_link">
-            <inertial>
-                <origin xyz="0.19104 -0.000401365 -0.0214358" rpy="0 0 0"/>
-                <mass value="2.10608"/>
-                <inertia ixx="0.00612771" ixy="-0.00148492" ixz="-0.000269689" iyy="0.0355118" iyz="-2.47513e-05" izz="0.0374813"/>
-            </inertial>
-            <!-- Part humerus_link_parts -->
-            <visual>
-                <origin xyz="0.19104 -0.000401365 -0.0214358" rpy="-2.48682 1.55043 -2.48996"/>
-                <geometry>
-                    <mesh filename="file://$(find umrt-project-perry-description)/assets/merged/humerus_link_visual.stl"/>
-                </geometry>
-                <material name="humerus_link_parts_material">
-                    <color rgba="0.470126 0.661547 0.742536 1"/>
-                </material>
-            </visual>
-            <collision>
-                <origin xyz="0.19104 -0.000401365 -0.0214358" rpy="-2.48682 1.55043 -2.48996"/>
-                <geometry>
-                    <mesh filename="file://$(find umrt-project-perry-description)/assets/merged/humerus_link_collision.stl"/>
-                </geometry>
-            </collision>
-        </link>
-        <!-- Link flat_pattern_of_humerus_link -->
-        <link name="flat_pattern_of_humerus_link">
-            <inertial>
-                <origin xyz="-0.00600861 -0.120661 0.0450797" rpy="0 0 0"/>
-                <mass value="2.41904"/>
-                <inertia ixx="0.0672327" ixy="0.0021158" ixz="-1.93671e-06" iyy="0.00894428" iyz="2.2352e-05" izz="0.064383"/>
-            </inertial>
-            <!-- Part flat_pattern_of_humerus_link_parts -->
-            <visual>
-                <origin xyz="-0.00600861 -0.120661 0.0450797" rpy="-2.48682 1.55043 0.651633"/>
-                <geometry>
-                    <mesh filename="file://$(find umrt-project-perry-description)/assets/merged/flat_pattern_of_humerus_link_visual.stl"/>
-                </geometry>
-                <material name="flat_pattern_of_humerus_link_parts_material">
-                    <color rgba="0.358759 0.586672 0.658794 1"/>
-                </material>
-            </visual>
-            <collision>
-                <origin xyz="-0.00600861 -0.120661 0.0450797" rpy="-2.48682 1.55043 0.651633"/>
-                <geometry>
-                    <mesh filename="file://$(find umrt-project-perry-description)/assets/merged/flat_pattern_of_humerus_link_collision.stl"/>
-                </geometry>
-            </collision>
-        </link>
-        <!-- Link wirst_body -->
-        <link name="wirst_body">
-            <inertial>
-                <origin xyz="1.74216e-05 -0.0133229 -0.0449775" rpy="0 0 0"/>
-                <mass value="0.114952"/>
-                <inertia ixx="0.000141143" ixy="-3.67177e-10" ixz="8.43247e-07" iyy="0.000208967" iyz="4.47572e-13" izz="9.77212e-05"/>
-            </inertial>
-            <!-- Part wirst_body_parts -->
-            <visual>
-                <origin xyz="1.74216e-05 -0.0133229 -0.0449775" rpy="-2.48682 1.55043 0.651633"/>
-                <geometry>
-                    <mesh filename="file://$(find umrt-project-perry-description)/assets/merged/wirst_body_visual.stl"/>
-                </geometry>
-                <material name="wirst_body_parts_material">
-                    <color rgba="0.0745098 0.678431 0.972549 1"/>
-                </material>
-            </visual>
-            <collision>
-                <origin xyz="1.74216e-05 -0.0133229 -0.0449775" rpy="-2.48682 1.55043 0.651633"/>
-                <geometry>
-                    <mesh filename="file://$(find umrt-project-perry-description)/assets/merged/wirst_body_collision.stl"/>
-                </geometry>
-            </collision>
-        </link>
-        <!-- Link wrist_link -->
+            <collision>
+                <origin xyz="0 0 ${height3/2 - axel_offset}" rpy="0 0 0"/>
+                <geometry>
+                    <box size="${width} ${width} ${height3}"/>
+                </geometry>
+            </collision>
+            <visual>
+                <origin xyz="0 0 ${height3/2 - axel_offset}" rpy="0 0 0"/>
+                <geometry>
+                    <box size="${width} ${width} ${height3}"/>
+                </geometry>
+                <material name="orange"/>
+            </visual>
+            <inertial>
+                <origin xyz="0 0 ${height3/2 - axel_offset}" rpy="0 0 0"/>
+                <mass value="${mass}"/>
+                <inertia
+                        ixx="${mass / 12.0 * (width*width + height3*height3)}" ixy="0.0" ixz="0.0"
+                        iyy="${mass / 12.0 * (height3*height3 + width*width)}" iyz="0.0"
+                        izz="${mass / 12.0 * (width*width + width*width)}"/>
+            </inertial>
+        </link>
+        <joint name="elbow_0_joint" type="revolute">
+            <parent link="humerus_link"/>
+            <child link="wrist_link"/>
+            <origin xyz="0 0 ${height3}" rpy="0 0 0"/>
+            <axis xyz="0 1 0"/>
+            <dynamics damping="0.7"/>
+            <limit lower="${-3*pi/4.0}" upper="${3*pi/4.0}" effort="100" velocity="1.0"/>
+        </joint>
+        <!-- Wrist Link -->
         <link name="wrist_link">
-            <inertial>
-                <origin xyz="-2.16903e-18 -4.83311e-17 -0.00183593" rpy="0 0 0"/>
-                <mass value="0.0230672"/>
-                <inertia ixx="6.54736e-06" ixy="-2.51728e-23" ixz="-4.00656e-23" iyy="6.54736e-06" iyz="-5.94725e-24" izz="1.27521e-05"/>
-            </inertial>
-            <!-- Part wrist_link_parts -->
-            <visual>
-                <origin xyz="-2.1684e-18 0 -0.00183593" rpy="-1.56756 -0.0123485 -0.0161902"/>
-                <geometry>
-                    <mesh filename="file://$(find umrt-project-perry-description)/assets/merged/wrist_link_visual.stl"/>
-                </geometry>
-                <material name="wrist_link_parts_material">
-                    <color rgba="0.972549 0.529412 0.00392157 1"/>
-                </material>
-            </visual>
-            <collision>
-                <origin xyz="-2.1684e-18 0 -0.00183593" rpy="-1.56756 -0.0123485 -0.0161902"/>
-                <geometry>
-                    <mesh filename="file://$(find umrt-project-perry-description)/assets/merged/wrist_link_collision.stl"/>
-                </geometry>
-            </collision>
-        </link>
-        <!-- Frame toolpoint (dummy link + fixed joint) -->
-        <link name="toolpoint">
-            <origin xyz="0 0 0" rpy="0 -0 0"/>
-            <inertial>
-                <origin xyz="0 0 0" rpy="0 0 0"/>
-                <mass value="1e-9"/>
-                <inertia ixx="0" ixy="0" ixz="0" iyy="0" iyz="0" izz="0"/>
-            </inertial>
-        </link>
-        <joint name="toolpoint_frame" type="fixed">
-            <origin xyz="6.01645e-15 -3.66374e-14 -0.185923" rpy="-2.31486e-13 -2.82334e-14 2.83915e-14"/>
+            <collision>
+                <origin xyz="0 0 ${height3/2 - axel_offset}" rpy="0 0 0"/>
+                <geometry>
+                    <box size="${width} ${width} ${height3}"/>
+                </geometry>
+            </collision>
+            <visual>
+                <origin xyz="0 0 ${height3/2 - axel_offset}" rpy="0 0 0"/>
+                <geometry>
+                    <box size="${width} ${width} ${height3}"/>
+                </geometry>
+                <material name="orange"/>
+            </visual>
+            <inertial>
+                <origin xyz="0 0 ${height3/2 - axel_offset}" rpy="0 0 0"/>
+                <mass value="${mass}"/>
+                <inertia
+                        ixx="${mass / 12.0 * (width*width + height3*height3)}" ixy="0.0" ixz="0.0"
+                        iyy="${mass / 12.0 * (height3*height3 + width*width)}" iyz="0.0"
+                        izz="${mass / 12.0 * (width*width + width*width)}"/>
+            </inertial>
+        </link>
+        <joint name="gripper_wrist_fixture" type="fixed">
             <parent link="wrist_link"/>
-            <child link="toolpoint"/>
-            <axis xyz="0 0 0"/>
-        </joint>
-        <!-- Joint from wirst_body to wrist_link -->
-        <joint name="wrist_roll" type="revolute">
-            <origin xyz="2.22045e-16 -0.0314483 -0.0449775" rpy="-1.5708 1.5708 0"/>
-            <parent link="wirst_body"/>
-            <child link="wrist_link"/>
-            <axis xyz="0 0 1"/>
-            <limit effort="10" velocity="10" lower="-3.141592653589793" upper="3.141592653589793"/>
-        </joint>
-        <!-- Joint from flat_pattern_of_humerus_link to wirst_body -->
-        <joint name="wrist_pitch" type="revolute">
-            <origin xyz="1.77636e-15 -0.3937 0.0899558" rpy="1.67261e-15 -2.51166e-15 -1.23947e-15"/>
-            <parent link="flat_pattern_of_humerus_link"/>
-            <child link="wirst_body"/>
-            <axis xyz="0 0 1"/>
-            <limit effort="10" velocity="10" lower="-1.5708" upper="1.5708"/>
-        </joint>
-        <!-- Joint from humerus_link to flat_pattern_of_humerus_link -->
-        <joint name="elbow_pitch" type="revolute">
-            <origin xyz="0.4572 0.031582 -0.067374" rpy="5.83832e-15 6.48493e-15 -3.14159"/>
-            <parent link="humerus_link"/>
-            <child link="flat_pattern_of_humerus_link"/>
-            <axis xyz="0 0 1"/>
-            <limit effort="10" velocity="10" lower="-0.610865" upper="0.959931"/>
-        </joint>
-        <!-- Joint from base_platter to humerus_link -->
-        <joint name="base_pitch" type="revolute">
-            <origin xyz="-0.0204961 -7.37257e-18 -0.0851182" rpy="-3.14159 1.5708 0"/>
-            <parent link="base_platter"/>
-            <child link="humerus_link"/>
-            <axis xyz="0 0 1"/>
-            <limit effort="10" velocity="10" lower="-1.5708" upper="1.5708"/>
-        </joint>
-        <!-- Joint from base_link to base_platter -->
-        <joint name="base_yaw" type="revolute">
-            <origin xyz="0.000390865 0.000967073 0.0809889" rpy="3.13835 -0.0161502 0.0124009"/>
-            <parent link="base_link"/>
-            <child link="base_platter"/>
-            <axis xyz="0 0 1"/>
-            <limit effort="10" velocity="10" lower="-3.141592653589793" upper="3.141592653589793"/>
-        </joint>
+            <child link="gripper_link"/>
+            <origin xyz="0 0 ${height3 - width}" rpy="0 0 0"/>
+        </joint>
+        <!-- Gripper Link -->
+        <link name="gripper_link">
+            <collision>
+                <origin xyz="0 0 ${gripper_thickness/2}" rpy="0 0 0"/>
+                <geometry>
+                    <box size="${gripper_width} ${gripper_breadth} ${gripper_thickness}"/>
+                </geometry>
+            </collision>
+            <visual>
+                <origin xyz="0 0 ${gripper_thickness/2}" rpy="0 0 0"/>
+                <geometry>
+                    <box size="${gripper_width} ${gripper_breadth} ${gripper_thickness}"/>
+                </geometry>
+                <material name="orange"/>
+            </visual>
+            <inertial>
+                <origin xyz="0 0 ${gripper_thickness/2}" rpy="0 0 0"/>
+                <mass value="${mass}"/>
+                <inertia
+                        ixx="${mass / 12.0 * (gripper_width*gripper_breadth + gripper_thickness*gripper_thickness)}" ixy="0.0" ixz="0.0"
+                        iyy="${mass / 12.0 * (gripper_thickness*gripper_thickness + gripper_width*gripper_breadth)}" iyz="0.0"
+                        izz="${mass / 12.0 * (gripper_width*gripper_breadth + gripper_width*gripper_breadth)}"/>
+            </inertial>
+        </link>
+        <joint name="gripper" type="prismatic">
+            <origin xyz="${-gripper_width/2 - width/2} 0 ${gripper_thickness}" rpy="0 0 0"/>
+            <parent link="gripper_link"/>
+            <child link="finger_left_link"/>
+            <axis xyz="1 0 0"/>
+            <dynamics damping="0.7"/>
+            <limit lower="0" upper="${gripper_width/2 - finger_thickness}" effort="100" velocity="1.0"/>
+        </joint>
+        <joint name="gripper_mimic" type="prismatic">
+            <origin xyz="${-gripper_width/2 - width/2} 0 ${gripper_thickness}" rpy="0 0 0"/>
+            <parent link="gripper_link"/>
+            <child link="finger_right_link"/>
+            <mimic joint="gripper" multiplier="-1" offset="0.5"/>
+            <axis xyz="1 0 0"/>
+            <dynamics damping="0.7"/>
+            <limit lower="${-gripper_width/2 + finger_thickness}" upper="0" effort="100" velocity="1.0"/>
+        </joint>
+        <!-- Finger Links -->
+        <link name="finger_left_link">
+            <collision>
+                <origin xyz="${finger_thickness*1.5} 0 ${finger_length/2}" rpy="0 0 0"/>
+                <geometry>
+                    <box size="${finger_thickness} ${gripper_breadth} ${finger_length}"/>
+                </geometry>
+            </collision>
+            <visual>
+                <origin xyz="${finger_thickness*1.5} 0 ${finger_length/2}" rpy="0 0 0"/>
+                <geometry>
+                    <box size="${finger_thickness} ${gripper_breadth} ${finger_length}"/>
+                </geometry>
+                <material name="orange"/>
+            </visual>
+            <inertial>
+                <origin xyz="${finger_thickness*1.5} 0 ${finger_length/2}" rpy="0 0 0"/>
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
Commit message: Replaced base_link IKFast works

File: ik2/project_perry_description.urdf.xacro (robot description, xacro)
@@ -26,25 +26,25 @@
         <!-- Base Link -->
         <link name="base_link">
-            <collision>
-                <origin xyz="0 0 ${base_height/2}" rpy="0 0 0"/>
-                <geometry>
-                    <box size="${base_width} ${base_width} ${base_height}"/>
-                </geometry>
-            </collision>
-            <visual>
-                <origin xyz="0 0 ${base_height/2}" rpy="0 0 0"/>
-                <geometry>
-                    <box size="${base_width} ${base_width} ${base_height}"/>
-                </geometry>
-                <material name="orange"/>
-            </visual>
-            <inertial>
-                <origin xyz="0 0 ${base_height/2}" rpy="0 0 0"/>
-                <mass value="${mass}"/>
-                <inertia
-                        ixx="${mass / 12.0 * (base_width*base_width + base_height*base_height)}" ixy="0.0" ixz="0.0"
-                        iyy="${mass / 12.0 * (base_height*base_height + base_width*base_width)}" iyz="0.0"
-                        izz="${mass / 12.0 * (base_width*base_width + base_width*base_width)}"/>
-            </inertial>
+            <inertial>
+                <origin xyz="0.00286812 -0.0209097 0.0286943" rpy="0 0 0"/>
+                <mass value="2.80632"/>
+                <inertia ixx="0.0231691" ixy="0.00065571" ixz="-0.000230556" iyy="0.0147789" iyz="0.000656447" izz="0.0344912"/>
+            </inertial>
+            <!-- Part base_link_parts -->
+            <visual>
+                <origin xyz="0.00286812 -0.0209097 0.0286943" rpy="0 -0 0"/>
+                <geometry>
+                    <mesh filename="file://$(find umrt-project-perry-description)/assets/merged/base_link_visual.stl"/>
+                </geometry>
+                <material name="base_link_parts_material">
+                    <color rgba="0.0745098 0.678431 0.972549 1"/>
+                </material>
+            </visual>
+            <collision>
+                <origin xyz="0.00286812 -0.0209097 0.0286943" rpy="0 -0 0"/>
+                <geometry>
+                    <mesh filename="file://$(find umrt-project-perry-description)/assets/merged/base_link_collision.stl"/>
+                </geometry>
+            </collision>
         </link>
         <joint name="base_yaw_joint" type="continuous">
